File: vco-100-200.kicad_sch (KiCad schematic)
At the start: 7 parts, among them J3 Conn_01x06_Pin

Commit message: Update pcb routing, add 50 Ohm net classes
Other:
- moved on the sheet: XS1, XS2
Changed lines of the file:
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@@
+	)
+	(junction
+		(at 57.15 68.58)
+		(diameter 0)
+		(color 0 0 0 0)
 	)
 	(junction
@@
 	(wire
 		(pts
+			(xy 57.15 68.58) (xy 67.31 68.58)
+		)
+		(stroke
+			(width 0)
+			(type default)
+		)
+	)
+	(wire
+		(pts
 			(xy 87.63 80.01) (xy 87.63 85.09)
 		)
@@
 	(wire
 		(pts
-			(xy 64.77 68.58) (xy 67.31 68.58)
+			(xy 54.61 68.58) (xy 57.15 68.58)
 		)
 		(stroke
@@
 	(wire
 		(pts
-			(xy 180.34 68.58) (xy 181.61 68.58)
+			(xy 57.15 66.04) (xy 57.15 68.58)
+		)
+		(stroke
+			(width 0)
+			(type default)
+		)
+	)
+	(wire
+		(pts
+			(xy 180.34 68.58) (xy 187.96 68.58)
 		)
 		(stroke
@@
 			(width 0)
 			(type default)
+		)
+	)
+	(netclass_flag ""
+		(length 2.54)
+		(shape round)
+		(at 124.46 63.5 0)
+		(fields_autoplaced yes)
+		(effects
+			(font
+				(size 1.27 1.27)
+			)
+			(justify left bottom)
+		)
+		(property "Netclass" "50 Ohm"
+			(at 125.1585 60.96 0)
+			(effects
+				(font
+					(size 1.27 1.27)
+				)
+				(justify left)
+			)
+		)
+		(property "Component Class" ""
+			(at 38.1 -6.35 0)
+			(effects
+				(font
+					(size 1.27 1.27)
+					(italic yes)
+				)
+			)
+		)
+	)
+	(netclass_flag ""
+		(length 2.54)
+		(shape round)
+		(at 57.15 66.04 0)
+		(fields_autoplaced yes)
+		(effects
+			(font
+				(size 1.27 1.27)
+			)
+			(justify left bottom)
+		)
+		(property "Netclass" "50 Ohm"
+			(at 57.8485 63.5 0)
+			(effects
+				(font
+					(size 1.27 1.27)
+				)
+				(justify left)
+			)
+		)
+		(property "Component Class" ""
+			(at -29.21 -3.81 0)
+			(effects
+				(font
+					(size 1.27 1.27)
+					(italic yes)
+				)
+			)
+		)
+	)
+	(netclass_flag ""
+		(length 2.54)
+		(shape round)
+		(at 184.15 68.58 0)
+		(fields_autoplaced yes)
+		(effects
+			(font
+				(size 1.27 1.27)
+			)
+			(justify left bottom)
+		)
+		(property "Netclass" "50 Ohm"
+			(at 184.8485 66.04 0)
+			(effects
+				(font
+					(size 1.27 1.27)
+				)
+				(justify left)
+			)
+		)
+		(property "Component Class" ""
+			(at 97.79 -1.27 0)
+			(effects
+				(font
+					(size 1.27 1.27)
+					(italic yes)
+				)
+			)
 		)
 	)
 	(symbol
 		(lib_id "connectors:RF-PCB-pin-place")
-		(at 185.42 68.58 0)
+		(at 191.77 68.58 0)
 		(unit 1)
 		(exclude_from_sim no)
@@
 		(fields_autoplaced yes)
 		(property "Reference" "XS1"
-			(at 185.42 65.278 0)
+			(at 191.77 65.278 0)
 			(do_not_autoplace yes)
 			(effects
@@
 		)
 		(property "Value" "~"
-			(at 185.42 68.58 0)
+			(at 191.77 68.58 0)
 			(effects
 				(font
@@
 		)
 		(property "Footprint" "RF-connectors:RF-PCB-pin-place"
-			(at 185.42 68.58 0)
+			(at 191.77 68.58 0)
 			(effects
 				(font
@@
 		)
 		(property "Datasheet" ""
-			(at 185.42 68.58 0)
+			(at 191.77 68.58 0)
 			(effects
 				(font
@@
 		)
 		(property "Description" "PCB pin soldering place for the housing places SMA connectors"
-			(at 185.42 68.58 0)
+			(at 191.77 68.58 0)
 			(effects
 				(font
@@
 		)
 		(property "Partnumber" ""
-			(at 185.42 68.58 0)
+			(at 191.77 68.58 0)
 			(effects
 				(font
@@
 	(symbol
 		(lib_id "connectors:RF-PCB-pin-place")
-		(at 60.96 68.58 0)
+		(at 50.8 68.58 0)
 		(mirror y)
 		(unit 1)
@@
 		(dnp no)
 		(property "Reference" "XS2"
-			(at 60.96 65.278 0)
+			(at 50.8 65.278 0)
 			(do_not_autoplace yes)
 			(effects
@@
 		)
 		(property "Value" "~"
-			(at 60.96 68.58 0)
+			(at 50.8 68.58 0)
 			(effects
 				(font
@@
 		)
 		(property "Footprint" "RF-connectors:RF-PCB-pin-place"
-			(at 60.96 68.58 0)
+			(at 50.8 68.58 0)
 			(effects
 				(font
@@
 		)
 		(property "Datasheet" ""
-			(at 60.96 68.58 0)
+			(at 50.8 68.58 0)
 			(effects
 				(font
@@
 		)
 		(property "Description" "PCB pin soldering place for the housing places SMA connectors"
-			(at 60.96 68.58 0)
+			(at 50.8 68.58 0)
 			(effects
 				(font
@@
 		)
 		(property "Partnumber" ""
-			(at 60.96 68.58 0)
+			(at 50.8 68.58 0)
 			(effects
 				(font
@@
 	(symbol
 		(lib_id "power:Earth")
-		(at 60.96 71.12 0)
+		(at 50.8 71.12 0)
 		(unit 1)
 		(exclude_from_sim no)
@@
 		(fields_autoplaced yes)
 		(property "Reference" "#PWR012"
-			(at 60.96 77.47 0)
+			(at 50.8 77.47 0)
 			(effects
 				(font
@@
 		)
 		(property "Value" "Earth"
-			(at 60.96 76.2 0)
+			(at 50.8 76.2 0)
 			(effects
 				(font
@@
 		)
 		(property "Footprint" ""
-			(at 60.96 71.12 0)
+			(at 50.8 71.12 0)
 			(effects
 				(font
@@
 		)
 		(property "Datasheet" "~"
-			(at 60.96 71.12 0)
+			(at 50.8 71.12 0)
 			(effects
 				(font
@@
 		)
 		(property "Description" "Power symbol creates a global label with name \"Earth\""
-			(at 60.96 71.12 0)
+			(at 50.8 71.12 0)
 			(effects
 				(font
@@
 	(symbol
 		(lib_id "power:Earth")
-		(at 185.42 71.12 0)
+		(at 191.77 71.12 0)
 		(unit 1)
 		(exclude_from_sim no)
@@
 		(fields_autoplaced yes)
 		(property "Reference" "#PWR010"
-			(at 185.42 77.47 0)
+			(at 191.77 77.47 0)
 			(effects
 				(font
@@
 		)
 		(property "Value" "Earth"
-			(at 185.42 76.2 0)
+			(at 191.77 76.2 0)
 			(effects
 				(font
@@
 		)
 		(property "Footprint" ""
-			(at 185.42 71.12 0)
+			(at 191.77 71.12 0)
 			(effects
 				(font
@@
 		)
 		(property "Datasheet" "~"
-			(at 185.42 71.12 0)
+			(at 191.77 71.12 0)
 			(effects
 				(font
@@
 		)
 		(property "Description" "Power symbol creates a global label with name \"Earth\""
-			(at 185.42 71.12 0)
-			(effects
-				(font
+			(at 191.77 71.12 0)
+			(effects
+				(font
